File: FlightControllerHardware/FlightControllerHardware.kicad_sch (KiCad schematic)
At the start: 21 parts, among them J1 Power in, J2 Power in, J3 servoRight, J4 servoBack, J5 servoLeft, J6 servoFront, J7 mainThrust, SW1 SW_Push, U1 module_bme280, U2 Pico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

Commit message: finished routing
Parts:
- added J3: Conn_01x20_Male, Connector_PinHeader_2.54mm:PinHeader_1x20_P2.54mm_Vertical, symbol Connector:Conn_01x20_Male
- renumbered J3 to J4, J4 to J5, J5 to J6, J6 to J7, J7 to J8
Connections:
- net +3V3: now also J3.16 (Pin_16)
- net GND: no longer U2.13 (GND)
- net gpsRx: now also U2.21 (GPIO16), J3.1 (Pin_1); no longer U2.1 (GPIO0)
- net gpsTx: now also U2.22 (GPIO17), J3.2 (Pin_2); no longer U2.2 (GPIO1)
- net at U2.23 (GND): now also J3.3 (Pin_3)
- net at U2.24 (GPIO18): now also J3.4 (Pin_4)
- net at U2.25 (GPIO19): now also J3.5 (Pin_5)
- net at U2.26 (GPIO20): now also J3.6 (Pin_6)
- net at U2.27 (GPIO21): now also J3.7 (Pin_7)
- net at SW1.2, U2.28 (GND): now also J3.8 (Pin_8)
- net at U2.29 (GPIO22): now also J3.9 (Pin_9)
- net at SW1.1, U2.30 (RUN): now also J3.10 (Pin_10)
- net at U2.31 (GPIO26_ADC0): now also J3.11 (Pin_11)
- net at U2.32 (GPIO27_ADC1): now also J3.12 (Pin_12)
- net at U2.33 (AGND): now also J3.13 (Pin_13)
- net at U2.34 (GPIO28_ADC2): now also J3.14 (Pin_14)
- net at U2.35 (ADC_VREF): now also J3.15 (Pin_15)
- net at U2.37 (3V3_EN): now also J3.17 (Pin_17)
- net at U2.38 (GND): now also J3.18 (Pin_18)
- net at U2.39 (VSYS): now also J3.19 (Pin_19)
- net at U2.40 (VBUS): now also J3.20 (Pin_20)
- no-connect marks 32 -> 18
Other:
- moved on the sheet: SW1
